File: pcb/proj.kicad_sch (KiCad schematic)
At the start: 106 parts, among them J1 Conn_01x04, SW1 SW_Push, SW10 8, SW11 9, SW12 /, SW13 SW_Push, SW14 SW_Push, SW15 4, SW16 5, SW17 6, SW18 X, SW19 SW_Push, SW2 SW_Push, SW20 SW_Push, SW21 1, SW22 2, SW23 3, SW24 -, SW25 Alpha, SW26 SW_Push, SW27 SW_Push, SW28 SW_Push, SW29 SW_Push, SW3 ., SW30 +, SW31 2nd, SW32 SW_Push, SW33 SW_Push, SW34 SW_Push, SW35 SW_Push, SW36 SW_Push, SW37 Graph, SW38 Programs, SW39 Left, SW4 0, SW40 Up, SW41 Right, SW42 Down, SW43 Power, SW44 Reset, SW5 +/-, SW6 =, SW7 SW_Push, SW8 SW_Push, SW9 7, U1 PIC16C74, U2 STM32F401RCTx, U3 74HC138, U4 LTC3525-5, Y1 20MHz

Commit message: fix
Parts:
- U3: value 74HC138 -> 74HC238
Changed lines of the file:
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@@
 			)
 		)
-		(property "Value" "74HC138"
+		(property "Value" "74HC238"
 			(at 131.572 40.386 0)
 			(effects

Commit message: work
Parts:
- SW13: value SW_Push -> Deg/Rad
- SW19: value SW_Push -> Constants
- SW26: value SW_Push -> (/)
- SW27: value SW_Push -> Sin(x)/Sin-1(x)
- SW28: value SW_Push -> Cos(x)/Cos-1(x)
- SW29: value SW_Push -> Tan(x)/Tan-1(x)
- SW32: value SW_Push -> Γ(x)/
- SW33: value SW_Push -> x^y/y√x
- SW34: value SW_Push -> x^2/√x
- SW35: value SW_Push -> log(x)/ln(x)
- SW36: value SW_Push -> e^x/10^x
- SW7: value SW_Push -> Sci/Norm
Changed lines of the file:
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@@
 			)
 		)
-		(property "Value" "SW_Push"
+		(property "Value" "Γ(x)/"
 			(at 200.66 62.484 0)
 			(effects
@@
 			)
 		)
-		(property "Value" "SW_Push"
+		(property "Value" "x^2/√x"
 			(at 256.54 62.484 0)
 			(effects
@@
 			)
 		)
-		(property "Value" "SW_Push"
+		(property "Value" "x^y/y√x"
 			(at 228.6 62.484 0)
 			(effects
@@
 			)
 		)
-		(property "Value" "SW_Push"
+		(property "Value" "(/)"
 			(at 200.66 53.594 0)
 			(effects
@@
 			)
 		)
-		(property "Value" "SW_Push"
+		(property "Value" "Deg/Rad"
 			(at 172.72 35.814 0)
 			(effects
@@
 			)
 		)
-		(property "Value" "SW_Push"
+		(property "Value" "Sci/Norm"
 			(at 172.72 26.924 0)
 			(effects
@@
 			)
 		)
-		(property "Value" "SW_Push"
+		(property "Value" "Sin(x)/Sin-1(x)"
 			(at 228.6 53.594 0)
 			(effects
@@
 			)
 		)
-		(property "Value" "SW_Push"
+		(property "Value" "log(x)/ln(x)"
 			(at 284.48 62.484 0)
 			(effects
@@
 			)
 		)
-		(property "Value" "SW_Push"
+		(property "Value" "e^x/10^x"
 			(at 312.42 62.484 0)
 			(effects
@@
 			)
 		)
-		(property "Value" "SW_Push"
+		(property "Value" "Constants"
 			(at 172.72 44.704 0)
 			(effects
@@
 			)
 		)
-		(property "Value" "SW_Push"
+		(property "Value" "Tan(x)/Tan-1(x)"
 			(at 284.48 53.594 0)
 			(effects
@@
 			)
 		)
-		(property "Value" "SW_Push"
+		(property "Value" "Cos(x)/Cos-1(x)"
 			(at 256.54 53.594 0)
 			(effects

Commit message: work
Parts:
- added D43: 2nd, LED_THT:LED_D5.0mm, symbol Device:LED
- added D44: Alpha, LED_THT:LED_D5.0mm, symbol Device:LED
- added D45: Deg, LED_THT:LED_D5.0mm, symbol Device:LED
- added D46: Rad, LED_THT:LED_D5.0mm, symbol Device:LED
- added R1, R2, R3, R4: 470Ω, Resistor_THT:R_Axial_DIN0207_L6.3mm_D2.5mm_P10.16mm_Horizontal, symbol Device:R_US
- SW1: value SW_Push -> Reset
- SW14: value SW_Push -> Clear
- SW2: value SW_Push -> Y/Stats
- SW20: value SW_Push -> Del
- SW3: value . -> ./,
- SW32: value Γ(x)/ -> Γ(x)
- SW6: value = -> Solve/=
- SW8: value SW_Push -> X/Matrix
- U3: symbol 74xx:74HC138 -> 74xx:74HC238
Connections:
- net GND: now also D43.1 (K), D44.1 (K), D45.1 (K), D46.1 (K)
- net 2ND: now reaches U1.19 (RD0/PSP0)
- net 2ND: now also R1.1
- net ALPHA: now reaches U1.20 (RD1/PSP1)
- net ALPHA: now also R2.1
- net RAD: now reaches U1.21 (RD2/PSP2)
- net RAD: now also R4.1
- net DEG: now reaches U1.22 (RD3/PSP3)
- net DEG: now also R3.1
- new net: D45.2 (A), R3.2
- new net: D44.2 (A), R2.2
- new net: D46.2 (A), R4.2
- new net: D43.2 (A), R1.2
- no-connect marks 76 -> 72
