File: pcb/proj.kicad_sch (KiCad schematic)
At the start: 123 parts, among them J1 Conn_01x04, SW1 Reset, SW10 8, SW11 9, SW12 /, SW13 Deg/Rad, SW14 Clear, SW15 4, SW16 5, SW17 6, SW18 X, SW19 Constants, SW2 Y/Stats, SW20 Del, SW21 1, SW22 2, SW23 3, SW24 -, SW25 Alpha, SW26 (/), SW27 Sin(x)/Sin-1(x), SW28 Cos(x)/Cos-1(x), SW29 Tan(x)/Tan-1(x), SW3 ./,, SW30 +, SW31 2nd, SW32 Γ(x), SW33 x^y/y√x, SW34 x^2/√x, SW35 log(x)/ln(x), SW36 e^x/10^x, SW37 Graph, SW38 Programs, SW39 Left, SW4 0, SW40 Up, SW41 Right, SW42 Down, SW43 Power, SW44 FPU Reset, SW45 Main Reset, SW5 +/-, SW6 Solve/=, SW7 Sci/Norm, SW8 X/Matrix, SW9 7, U1 PIC16C74, U2 STM32F401RCTx, U3 74HC238, U4 LTC3525-5, Y1 20MHz

Commit message: work
Parts:
- removed U4: LTC3525-5, Package_TO_SOT_SMD:SOT-363_SC-70-6, symbol Regulator_Switching:LTC3525-5
- added U4: ISL9111EH50Z-T7A, Package_TO_SOT_SMD:SOT-23-6_Handsoldering, symbol symbols:ISL9111EH50Z-T7A
- C8: value 1µF -> 4.7µF
- C9: value 10µF -> 4.7µF; footprint Capacitor_THT:CP_Radial_D6.3mm_P2.50mm -> Capacitor_THT:CP_Radial_D5.0mm_P2.00mm
- L1: value 10µH -> 4.7µH; footprint Inductor_SMD:L_0805_2012Metric_Pad1.05x1.20mm_HandSolder -> Inductor_SMD:L_1008_2520Metric_Pad1.43x2.20mm_HandSolder
- R10, R6, R8: value 20kΩ -> 2kΩ; footprint (none) -> Resistor_SMD:R_1206_3216Metric_Pad1.30x1.75mm_HandSolder
- R11, R12: footprint (none) -> Resistor_SMD:R_1206_3216Metric_Pad1.30x1.75mm_HandSolder
- R5, R7, R9: value 10kΩ -> 1kΩ; footprint (none) -> Resistor_SMD:R_1206_3216Metric_Pad1.30x1.75mm_HandSolder
Connections:
- net +3.3V: now also U4.3 (EN), U4.6 (VIN)
- net +5V: now also U4.5 (VOUT)
- net GND: now also U4.2 (GND)
- net at L1.2: now also U4.1 (SW)
- no-connect marks 72 -> 73

Commit message: pcb work
Parts:
- added U5: SN74LVC1G32DBVR, Package_TO_SOT_SMD:SOT-23-5_HandSoldering, symbol symbols:SN74LVC1G32DBVR
Connections:
- net +5V: now also U5.5 (VCC)
- net DSS: now also U5.2
- net GND: now also U5.3 (GND)
- net SCK: now also U5.1; no longer DS1.6 (SCK)
- new net: DS1.6 (SCK), U5.4

Commit message: board
Parts:
- removed C7: 100nF, Capacitor_SMD:C_1206_3216Metric_Pad1.33x1.80mm_HandSolder, symbol Device:C
- removed J1: Conn_01x04, Connector_PinHeader_2.54mm:PinHeader_1x04_P2.54mm_Vertical, symbol Connector_Generic:Conn_01x04
- added J1: Conn_02x05_Odd_Even, Connector_IDC:IDC-Header_2x05_P2.54mm_Vertical, symbol Connector_Generic:Conn_02x05_Odd_Even
- added R13: 10kΩ, Resistor_SMD:R_1206_3216Metric_Pad1.30x1.75mm_HandSolder, symbol Device:R_US
- added RN1: 10kΩ, Resistor_THT:R_Array_SIP7, symbol Device:R_Network06_US
Connections:
- net +3.3V: now also SW44.2, J1.7 (Pin_7), J1.8 (Pin_8)
- net GND: now also J1.5 (Pin_5), J1.6 (Pin_6), R13.2, RN1.1 (common); no longer SW44.1, U2.60 (BOOT0)
- net at D12.1 (K), D18.1 (K), D24.1 (K)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: now also RN1.2 (R1)
- net at D1.1 (K), D13.1 (K), D19.1 (K)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: now also RN1.7 (R6)
- net at D15.1 (K), D21.1 (K), D27.1 (K)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: now also RN1.5 (R4)
- net FPURST: now reaches U2.7 (NRST)
- net FPURST: now also J1.1 (Pin_1); no longer SW44.2
- net SWDIO: now reaches U2.46 (PA13)
- net SWDIO: now also J1.4 (Pin_4)
- net SWCLK: now reaches U2.49 (PA14)
- net SWCLK: now also J1.2 (Pin_2)
- net at D14.1 (K), D2.1 (K), D20.1 (K)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: now also RN1.6 (R5)
- net at D10.1 (K), D16.1 (K), D22.1 (K)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: now also RN1.4 (R3)
- net at D11.1 (K), D17.1 (K), D23.1 (K)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: now also RN1.3 (R2)
- net SWO: now reaches U2.55 (PB3)
- net SWO: now also J1.3 (Pin_3)
- new net: R13.1, SW44.1, U2.60 (BOOT0)
- no-connect marks 73 -> 74
Other:
- moved on the sheet: R11, SW44

Commit message: Fixes
Parts:
- SW44: value FPU Reset -> FPU BOOT0
- SW45: value Main Reset -> Reset
- renumbered C8 to C7, C9 to C8
Connections:
- net +5V: now also DS1.4 (CS)
- net DSS: no longer DS1.4 (~{CS})
Changed lines of the file:
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@@
 	)
 	(junction
+		(at 54.61 135.89)
+		(diameter 0)
+		(color 0 0 0 0)
+	)
+	(junction
 		(at 130.81 95.25)
 		(diameter 0)
@@
 	(wire
 		(pts
+			(xy 54.61 135.89) (xy 71.12 135.89)
+		)
+		(stroke
+			(width 0)
+			(type default)
+		)
+	)
+	(wire
+		(pts
 			(xy 99.06 41.91) (xy 99.06 54.61)
 		)
@@
 	(wire
 		(pts
+			(xy 54.61 135.89) (xy 54.61 147.32)
+		)
+		(stroke
+			(width 0)
+			(type default)
+		)
+	)
+	(wire
+		(pts
 			(xy 41.91 59.69) (xy 30.48 59.69)
 		)
@@
 	(wire
 		(pts
-			(xy 45.72 135.89) (xy 71.12 135.89)
+			(xy 45.72 135.89) (xy 54.61 135.89)
 		)
 		(stroke
@@
 	(global_label "DSS"
 		(shape input)
-		(at 54.61 147.32 180)
-		(fields_autoplaced yes)
-		(effects
-			(font
-				(size 1.27 1.27)
-			)
-			(justify right)
-		)
-		(property "Intersheetrefs" "${INTERSHEET_REFS}"
-			(at 47.9358 147.32 0)
-			(effects
-				(font
-					(size 1.27 1.27)
-				)
-				(justify right)
-				(hide yes)
-			)
-		)
-	)
-	(global_label "DSS"
-		(shape input)
 		(at 105.41 54.61 0)
 		(fields_autoplaced yes)
@@
 			)
 		)
-		(property "Value" "FPU Reset"
+		(property "Value" "FPU BOOT0"
 			(at 120.904 128.27 0)
 			(effects
@@
 		(on_board yes)
 		(dnp no)
-		(property "Reference" "C8"
+		(property "Reference" "C7"
 			(at 255.524 142.24 0)
 			(effects
@@
 			(project "proj"
 				(path "/9b3fd51f-0cc8-4d93-a874-8128b084ae71"
-					(reference "C8")
+					(reference "C7")
 					(unit 1)
 				)
@@
 			)
 		)
-		(property "Value" "Main Reset"
+		(property "Value" "Reset"
 			(at 34.544 35.56 0)
 			(effects
@@
 		(on_board yes)
 		(dnp no)
-		(property "Reference" "C9"
+		(property "Reference" "C8"
 			(at 302.514 142.24 0)
 			(effects
@@
 			(project "proj"
 				(path "/9b3fd51f-0cc8-4d93-a874-8128b084ae71"
-					(reference "C9")
+					(reference "C8")
 					(unit 1)
 				)
