File: pcb/proj.kicad_pcb (KiCad board)
At the start: 2 copper layers, 125 x 185 mm, 115 parts, among them J1 Conn_01x04, SW1 Reset, SW10 8, SW11 9, SW12 /, SW13 Deg/Rad, SW14 Clear, SW15 4, SW16 5, SW17 6, SW18 X, SW19 Constants, SW2 Y/Stats, SW20 Del, SW21 1, SW22 2, SW23 3, SW24 -, SW25 Alpha, SW26 (/), SW27 Sin(x)/Sin-1(x), SW28 Cos(x)/Cos-1(x), SW29 Tan(x)/Tan-1(x), SW3 ./,, SW30 +, SW31 2nd, SW32 Γ(x), SW33 x^y/y√x, SW34 x^2/√x, SW35 log(x)/ln(x), SW36 e^x/10^x, SW37 Graph, SW38 Programs, SW39 Left, SW4 0, SW40 Up, SW41 Right, SW42 Down, SW43 Power, SW44 FPU Reset, SW45 Main Reset, SW5 +/-, SW6 Solve/=, SW7 Sci/Norm, SW8 X/Matrix, SW9 7, U1 PIC16C74, U2 STM32F401RCTx, U3 74HC238, U4 LTC3525-5, Y1 20MHz

Commit message: work
Parts:
- added R10: 2kΩ, Resistor_SMD:R_1206_3216Metric_Pad1.30x1.75mm_HandSolder, F.Cu at (165.4, 100.4)
- added R11: 10kΩ, Resistor_SMD:R_1206_3216Metric_Pad1.30x1.75mm_HandSolder, F.Cu at (165.4, 103.7)
- added R12: 10kΩ, Resistor_SMD:R_1206_3216Metric_Pad1.30x1.75mm_HandSolder, F.Cu at (165.4, 107.0)
- added R5: 1kΩ, Resistor_SMD:R_1206_3216Metric_Pad1.30x1.75mm_HandSolder, F.Cu at (165.4, 84.0)
- added R6: 2kΩ, Resistor_SMD:R_1206_3216Metric_Pad1.30x1.75mm_HandSolder, F.Cu at (165.4, 87.3)
- added R7: 1kΩ, Resistor_SMD:R_1206_3216Metric_Pad1.30x1.75mm_HandSolder, F.Cu at (165.4, 90.5)
- added R8: 2kΩ, Resistor_SMD:R_1206_3216Metric_Pad1.30x1.75mm_HandSolder, F.Cu at (165.4, 93.8)
- added R9: 1kΩ, Resistor_SMD:R_1206_3216Metric_Pad1.30x1.75mm_HandSolder, F.Cu at (165.4, 97.1)
- C8: value 1µF -> 4.7µF
- C9: value 10µF -> 4.7µF; footprint Capacitor_THT:CP_Radial_D6.3mm_P2.50mm -> Capacitor_THT:CP_Radial_D5.0mm_P2.00mm
- L1: value 10µH -> 4.7µH; footprint Inductor_SMD:L_0805_2012Metric_Pad1.05x1.20mm_HandSolder -> Inductor_SMD:L_1008_2520Metric_Pad1.43x2.20mm_HandSolder
- U4: value LTC3525-5 -> ISL9111EH50Z-T7A; footprint Package_TO_SOT_SMD:SOT-363_SC-70-6 -> Package_TO_SOT_SMD:SOT-23-6_Handsoldering
- moved C9 12.3 mm to (147.8, 113.2)
- moved L1 7.12 mm to (143.5, 109.0), turned to 180 degrees
- moved C8 4.64 mm to (147.8, 106.8)
- moved U4 0.50 mm to (143.2, 114.0)
Connections:
- SW45 pad 2: Net-(R12-Pad2) -> Net-(U1-~{MCLR}/Vpp)
- U1 pad 1: +5V -> Net-(U1-~{MCLR}/Vpp)
- U4 pad 1: +3.3V -> Net-(U4-SW)
- U4 pad 4: +5V -> unconnected-(U4-~{FAULT}-Pad4)
- U4 pad 5: GND -> +5V
- U4 pad 6: Net-(U4-SW) -> +3.3V
Routing:
- net +5V: track 246.7 -> 57.3 mm, vias 2 -> 0
- net +3.3V: track 51.7 -> 34.7 mm
- net Net-(U4-SW): track 12.4 -> 0.00 mm
- net GND: track 52.7 -> 50.8 mm
- added copper zone on B.Cu, net +5V
- removed copper zone on B.Cu, net +3.3V

Commit message: pcb work
Parts:
- added U5: SN74LVC1G32DBVR, Package_TO_SOT_SMD:SOT-23-5_HandSoldering, F.Cu at (118.9, 39.0)
- moved R11 99.0 mm to (124.8, 13.5)
- moved R12 96.7 mm to (140.8, 13.5)
- moved R7 26.4 mm to (139.3, 87.2)
- moved R8 26.3 mm to (139.2, 93.0)
- moved R6 21.4 mm to (144.8, 93.0)
- moved R5 21.0 mm to (144.7, 87.2)
- moved R9 17.9 mm to (150.5, 87.2)
- moved R10 16.6 mm to (150.6, 93.0)
- moved C8 5.17 mm to (142.6, 106.5)
- moved C9 5.17 mm to (142.6, 113.0)
- moved L1 5.17 mm to (138.3, 108.8)
- moved U4 5.17 mm to (138.1, 113.8)
Connections:
- DS1 pad 6: SCK -> Net-(DS1-SCK)
Routing:
- net COSS: track 53.7 -> 49.7 mm
- net MOSI: track 128.5 -> 126.2 mm

Commit message: work
Parts:
- moved U5 20.5 mm to (119.2, 59.5)
Routing:
- net +3.3V: track 34.7 -> 161.2 mm, vias 4 -> 10
- net Net-(DS1-SCK): track 0.00 -> 81.6 mm, vias 0 -> 2
- net Net-(U1-~{MCLR}/Vpp): track 0.00 -> 69.9 mm, vias 0 -> 3
- net SCK: track 115.2 -> 48.3 mm
- net DSS: track 72.0 -> 137.1 mm, vias 0 -> 2
- net Net-(U2-PA7): track 0.00 -> 32.5 mm, vias 0 -> 2
- net Net-(U2-PA4): track 0.00 -> 25.2 mm, vias 0 -> 2
- net Net-(U2-PA5): track 0.00 -> 20.2 mm, vias 0 -> 2
- net MOSI: track 126.2 -> 145.5 mm
- net COSS: track 49.7 -> 66.7 mm
- net +5V: track 57.3 -> 63.2 mm, vias 0 -> 5
- net Net-(U4-SW): track 0.00 -> 4.23 mm
- net MISO: track 28.9 -> 27.2 mm

Commit message: board
Parts:
- removed C7: 100nF, Capacitor_SMD:C_1206_3216Metric_Pad1.33x1.80mm_HandSolder
- added R13: 10kΩ, Resistor_SMD:R_1206_3216Metric_Pad1.30x1.75mm_HandSolder, F.Cu at (148.5, 69.0)
- added RN1: 10kΩ, Resistor_THT:R_Array_SIP7, F.Cu at (119.5, 29.8)
- J1: value Conn_01x04 -> Conn_02x05_Odd_Even; footprint Connector_PinHeader_2.54mm:PinHeader_1x04_P2.54mm_Vertical -> Connector_IDC:IDC-Header_2x05_P2.54mm_Vertical
- moved J1 108.1 mm to (131.8, 182.0), turned to 90 degrees
Connections:
- J1 pad 1: +3.3V -> FPURST
- J1 pad 2: GND -> SWCLK
- J1 pad 3: Net-(J1-Pin_3) -> SWO
- J1 pad 4: Net-(J1-Pin_4) -> SWDIO
- SW44 pad 1: GND -> Net-(U2-BOOT0)
- SW44 pad 2: Net-(U2-NRST) -> +3.3V
- U2 pad 46: Net-(J1-Pin_3) -> SWDIO
- U2 pad 49: Net-(J1-Pin_4) -> SWCLK
- U2 pad 55: unconnected-(U2-PB3-Pad55) -> SWO
- U2 pad 60: GND -> Net-(U2-BOOT0)
- U2 pad 7: Net-(U2-NRST) -> FPURST
Routing:
- net SWO: track 0.00 -> 134.1 mm, vias 0 -> 1
- net SWDIO: track 0.00 -> 128.2 mm, vias 0 -> 1
- net SWCLK: track 0.00 -> 127.1 mm, vias 0 -> 1
- net +3.3V: track 161.2 -> 282.0 mm, vias 10 -> 11
- net FPURST: track 0.00 -> 111.6 mm, vias 0 -> 2
- net Net-(U2-NRST): track 39.6 -> 0.00 mm
- net Net-(U2-BOOT0): track 0.00 -> 36.7 mm
- net Net-(D14-K): track 374.0 -> 400.8 mm
- net Net-(J1-Pin_3): track 22.2 -> 0.00 mm
- net Net-(J1-Pin_4): track 21.8 -> 0.00 mm, vias 1 -> 0
- net Net-(D1-K): track 394.7 -> 413.9 mm, vias 1 -> 2
- net Net-(D11-K): track 357.2 -> 366.7 mm
- net Net-(D12-K): track 335.4 -> 343.6 mm, vias 1 -> 2
- net Net-(D10-K): track 372.3 -> 380.2 mm
- net Net-(D15-K): track 378.2 -> 384.4 mm
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
Commit message: Fixes
Parts:
- removed C9: 4.7µF, Capacitor_THT:CP_Radial_D5.0mm_P2.00mm
- added C7: 4.7µF, Capacitor_THT:CP_Radial_D5.0mm_P2.00mm, F.Cu at (142.5, 106.5)
- SW44: value FPU Reset -> FPU BOOT0
- SW45: value Main Reset -> Reset
- moved C3 30.3 mm to (121.0, 49.2), turned to 0 degrees
- moved R11 7.42 mm to (119.5, 18.8), turned to -90 degrees
- moved C8 6.50 mm to (142.6, 113.0)
Connections:
- C8 pad 1: +3.3V -> +5V
- DS1 pad 4: DSS -> +5V
Routing:
- net DSS: track 138.3 -> 60.0 mm
- net +5V: track 63.2 -> 88.5 mm, vias 5 -> 4
- net GND: track 48.2 -> 53.3 mm
- net Net-(U1-CVref/Vref-/AN2/RA2): track 72.4 -> 73.3 mm
- net Net-(U1-AN0/RA0): track 71.5 -> 72.3 mm
- net Net-(U1-AN1/RA1): track 72.4 -> 73.3 mm
