File: pcb/proj.kicad_pcb (KiCad board)
At the start: 2 copper layers, 125 x 185 mm, 130 parts, among them J1 Conn_02x05_Odd_Even, Q1 MMBT3904, SW1 Reset, SW10 8, SW11 9, SW12 /, SW13 Deg/Rad, SW14 Clear, SW15 4, SW16 5, SW17 6, SW18 X, SW19 Constants, SW2 Y/Stats, SW20 Del, SW21 1, SW22 2, SW23 3, SW24 -, SW25 Alpha, SW26 (/), SW27 Sin(x)/Sin-1(x), SW28 Cos(x)/Cos-1(x), SW29 Tan(x)/Tan-1(x), SW3 ./,, SW30 +, SW31 2nd, SW32 Γ(x), SW33 x^y/y√x, SW34 x^2/√x, SW35 log(x)/ln(x), SW36 e^x/10^x, SW37 Graph, SW38 Programs, SW39 Left, SW4 0, SW40 Up, SW41 Right, SW42 Down, SW43 Power, SW44 FPU BOOT0, SW45 Reset, SW5 +/-, SW6 Solve/=, SW7 Sci/Norm, SW8 X/Matrix, SW9 7, U1 PIC16C74, U2 STM32F401RCTx, U3 74HC238, U4 ISL9111EH50Z-T7A, U5 SN74LVC1G32DBVR, U8 SN74LV1T34DBV, Y1 20MHz

Commit message: work on v1.5
Parts:
- removed C3, C4, C5, C6: 100nF, Capacitor_SMD:C_1206_3216Metric_Pad1.33x1.80mm_HandSolder
- added C11: 100nF, Capacitor_SMD:C_0402_1005Metric, F.Cu at (136.0, 85.3)
- added C12: 100nF, Capacitor_SMD:C_0402_1005Metric, F.Cu at (129.5, 85.3)
- added C13: 100nF, Capacitor_SMD:C_0402_1005Metric, F.Cu at (125.2, 80.0)
- added C14: 1μF, Capacitor_SMD:C_0603_1608Metric, F.Cu at (135.9, 87.8)
- added C15: 4.7μF, Capacitor_SMD:C_0603_1608Metric, F.Cu at (122.2, 105.0)
- added C16: 4.7μF, Capacitor_SMD:C_0603_1608Metric, F.Cu at (129.3, 104.5)
- added C17: 100nF, Capacitor_SMD:C_0402_1005Metric, F.Cu at (142.9, 38.9)
- added C18: 100nF, Capacitor_SMD:C_0402_1005Metric, F.Cu at (143.9, 22.5)
- added C19: 100nF, Capacitor_SMD:C_0402_1005Metric, F.Cu at (128.8, 88.9)
- added C20: 2.2μF, Capacitor_SMD:C_0603_1608Metric, F.Cu at (133.7, 86.2)
- added C21: 10μF, Capacitor_SMD:C_0603_1608Metric, F.Cu at (137.7, 179.6)
- added C22: 10μF, Capacitor_SMD:C_0603_1608Metric, F.Cu at (136.1, 111.0)
- added C23: 10pF, Capacitor_SMD:C_0402_1005Metric, F.Cu at (124.2, 111.5)
- added C24: 22μF, Capacitor_SMD:C_0603_1608Metric, F.Cu at (126.2, 114.0)
- added C25: 22μF, Capacitor_SMD:C_0603_1608Metric, F.Cu at (124.6, 114.0)
- added C26: 1μF, Capacitor_SMD:C_0603_1608Metric, F.Cu at (145.4, 43.5)
- added C27: 100nF, Capacitor_SMD:C_0402_1005Metric, F.Cu at (122.6, 44.0)
- added C28: 4.7μF, Capacitor_SMD:C_0603_1608Metric, F.Cu at (142.2, 114.6)
- added C29: 100nF, Capacitor_SMD:C_0402_1005Metric, F.Cu at (136.2, 115.0)
- added L2: 0.47µH, Inductor_SMD:L_Coilcraft_XxL4040, F.Cu at (132.7, 113.7)
- added R12: 316kΩ, Resistor_SMD:R_0402_1005Metric, F.Cu at (125.3, 111.5)
- added R16: 100kΩ, Resistor_SMD:R_0402_1005Metric, F.Cu at (126.4, 111.5)
- added U6: TPS61021A, Package_SON:Texas_DSG0008A_WSON-8-1EP_2x2mm_P0.5mm_EP0.9x1.6mm, F.Cu at (128.7, 112.3)
- added U7: SiP32510DT, Package_TO_SOT_SMD:TSOT-23-6, F.Cu at (139.2, 114.6)
- C1, C2: footprint Capacitor_SMD:C_1206_3216Metric_Pad1.33x1.80mm_HandSolder -> Capacitor_SMD:C_0603_1608Metric
- C10: footprint Capacitor_SMD:C_1206_3216Metric_Pad1.33x1.80mm_HandSolder -> Capacitor_SMD:C_0402_1005Metric
- C7, C8: value 4.7µF -> 100nF; footprint Capacitor_THT:CP_Radial_D5.0mm_P2.00mm -> Capacitor_SMD:C_0402_1005Metric
- C9: value 2.2μF -> 100nF; footprint Capacitor_SMD:C_1206_3216Metric_Pad1.33x1.80mm_HandSolder -> Capacitor_SMD:C_0402_1005Metric
- R10, R11, R13, R14, R15, R5, R6, R7, R8, R9: footprint Resistor_SMD:R_1206_3216Metric_Pad1.30x1.75mm_HandSolder -> Resistor_SMD:R_0603_1608Metric
- U3: footprint Package_DIP:DIP-16_W7.62mm_Socket_LongPads -> Package_SO:SOIC-16_3.9x9.9mm_P1.27mm
- moved C9 112.1 mm to (52.1, 13.9), turned to 180 degrees
- moved C10 51.9 mm to (120.5, 60.1)
- moved C8 44.4 mm to (129.0, 70.7)
- moved C7 32.1 mm to (139.8, 74.5), turned to -90 degrees
- moved R13 16.3 mm to (132.2, 70.5)
- moved L1 15.6 mm to (124.5, 101.5), turned to -90 degrees
- moved U4 14.7 mm to (125.7, 105.8)
- moved R11 10.9 mm to (122.5, 29.2)
- moved R10 7.80 mm to (143.6, 89.5), turned to -90 degrees
- moved R9 6.96 mm to (143.6, 86.3), turned to -90 degrees
- moved R6 4.57 mm to (141.9, 89.4), turned to -90 degrees
- moved U3 3.94 mm to (124.5, 92.9)
- moved R8 3.74 mm to (140.3, 89.4), turned to -90 degrees
- moved R5 2.90 mm to (141.9, 86.3), turned to -90 degrees
- moved R14 2.48 mm to (124.0, 82.2)
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Connections:
- C8 pad 1: +5V -> +3.3V
- C9 pad 1: Net-(U2-VCAP1) -> +5V
- DS1 pad 16: (no net) -> unconnected-(DS1-Pad16)
- R14 pad 1: GND -> +3.3V
- SW43 pad 1: Net-(B1-+) -> Net-(SW43-B)
- SW43 pad 2: +3.3V -> Net-(B1-+)
- SW43 pad 3: unconnected-(SW43-C-Pad3) -> GND
Routing:
- net +3.3V: track 277.5 -> 7.11 mm, vias 10 -> 2
- net Net-(SW43-B): track 0.00 -> 102.7 mm
- net +5V: track 71.2 -> 0.00 mm, vias 6 -> 0
- net Net-(D1-K): track 407.8 -> 378.3 mm, vias 2 -> 0
- net FPURST: track 197.5 -> 225.5 mm, vias 4 -> 8
- net DSS: track 60.0 -> 32.1 mm, vias 2 -> 0
- net GND: track 58.3 -> 31.0 mm, vias 6 -> 61
- net SWCLK: track 131.5 -> 156.8 mm, vias 1 -> 2
- net Net-(D14-K): track 393.7 -> 369.1 mm, vias 1 -> 0
- net SWO: track 138.8 -> 160.5 mm
- net Net-(D11-K): track 359.1 -> 339.3 mm
- net Net-(U1-AN0/RA0): track 72.3 -> 89.4 mm, vias 0 -> 4
- net Net-(U2-PA7): track 32.5 -> 17.2 mm
- net Net-(D10-K): track 372.4 -> 357.7 mm, vias 1 -> 0
- net Net-(D12-K): track 337.8 -> 323.2 mm, vias 2 -> 0
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- added copper zone on F.Cu, net +3.3V
- added copper zone on F.Cu, net +5V
- added copper zone on B.Cu, net GND
- added copper zone on F.Cu, net Net-(B1-+)
- added copper zone on F.Cu, net Net-(L2-Pad2)
- added copper zone on F.Cu, net Net-(U4-SW)
- added copper zone on F.Cu, net Net-(U6-EN)
- removed copper zone on B.Cu, net +5V
Other:
- board text added: "PICalculator v1.5 Designed by: Kyle Schmerge Max Pastushkov https://github.com/kpzip/PICalculator"
- board text removed: "PICalculator v1.4 Designed by: Kyle Schmerge Max Pastushkov https://github.com/kpzip/PICalculator"

Commit message: w
Parts:
- D1, D10, D11, D12, D13, D14, D15, D16, D17, D18, D19, D2, D20, D21, D22, D23, D24, D25, D26, D27, D28, D29, D3, D30, D31, D32, D33, D34, D35, D36, D37, D38, D39, D4, D40, D41, D42, D5, D6, D7, D8, D9: footprint Diode_SMD:D_1206_3216Metric_Pad1.42x1.75mm_HandSolder -> Diode_SMD:D_SOD-123F
Routing:
- net Net-(D11-K): track 339.3 -> 341.4 mm
- net Net-(D38-A): track 15.5 -> 17.2 mm
- net Net-(D41-A): track 14.9 -> 16.4 mm
- net Net-(D42-A): track 15.3 -> 16.7 mm
- net Net-(D15-K): track 364.1 -> 365.2 mm
- net Net-(D14-K): track 369.1 -> 370.0 mm
- net Net-(D10-K): track 357.7 -> 358.5 mm
- net Net-(D1-K): track 378.3 -> 379.1 mm
- net Net-(D12-K): track 323.2 -> 323.8 mm

Commit message: BOM improvements
Parts:
- added C30: 100nF, Capacitor_SMD:C_0402_1005Metric, F.Cu at (147.3, 27.9)
- added U9: SN74LV1T34DBV, Package_TO_SOT_SMD:SOT-23-5, F.Cu at (144.7, 27.2)
- D1, D10, D11, D12, D13, D14, D15, D16, D17, D18, D19, D2, D20, D21, D22, D23, D24, D25, D26, D27, D28, D29, D3, D30, D31, D32, D33, D34, D35, D36, D37, D38, D39, D4, D40, D41, D42, D5, D6, D7, D8, D9: value S040S2R0 -> SMD1200PL-TP
Connections:
- U1 pad 33: CORDY -> CORDY_5V
Routing:
- net CORDY: track 55.0 -> 65.3 mm, vias 3 -> 4
- net CORDY_5V: track 0.00 -> 9.10 mm
- net GND: track 31.0 -> 33.3 mm, vias 61 -> 64

Commit message: add famous quote
Other:
- board text added: "PIC"
- board text added: "alculator"
- board text added: "{dblquote}boosts [..] personal attractiveness and charisma{dblquote} -Prof. Loai Salem"
Changed lines of the file:
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@@
 		(layer "Edge.Cuts")
+	)
+	(gr_text "{dblquote}boosts [..] personal \nattractiveness and charisma{dblquote}\n-Prof. Loai Salem"
+		(at 130.95 101.9 0)
+		(layer "F.SilkS")
+		(effects
+			(font
+				(size 1 1)
+				(thickness 0.1)
+			)
+			(justify left bottom)
+		)
+	)
+	(gr_text "alculator"
+		(at 136.3 96.35 0)
+		(layer "F.SilkS")
+		(effects
+			(font
+				(size 1 1)
+				(thickness 0.1)
+			)
+			(justify left bottom)
+		)
+	)
+	(gr_text "PIC"
+		(at 130.95 96.7 0)
+		(layer "F.SilkS")
+		(effects
+			(font
+				(face "Arial Black")
+				(size 2 2)
+				(thickness 0.2)
+			)
+			(justify left bottom)
+		)
+		(render_cache "PIC" 0
+			(polygon
+				(pts
+					(xy 132.355304 94.363131) (xy 132.492612 94.395605) (xy 132.602919 94.445697) (xy 132.691085 94.51218)
+					(xy 132.76248 94.59746) (xy 132.814762 94.699617) (xy 132.847826 94.822075) (xy 132.859612 94.969403)
+					(xy 132.847006 95.119969) (xy 132.81138 95.246837) (xy 132.75451 95.35438) (xy 132.676064 95.445799)
+					(xy 132.580346 95.516342) (xy 132.45924 95.569865) (xy 132.307033 95.604776) (xy 132.116625 95.617501)
+					(xy 131.781646 95.617501) (xy 131.781646 96.36) (xy 131.152233 96.36) (xy 131.152233 95.203265)
+					(xy 131.781646 95.203265) (xy 131.929413 95.203265) (xy 132.047042 95.194781) (xy 132.126422 95.173135)
+					(xy 132.178053 95.142327) (xy 132.21776 95.097695) (xy 132.241193 95.046498) (xy 132.249249 94.9865)
+					(xy 132.242222 94.927357) (xy 132.221764 94.875738) (xy 132.187456 94.829818) (xy 132.141322 94.797432)
+					(xy 132.067358 94.774619) (xy 131.95396 94.765582) (xy 131.781646 94.765582) (xy 131.781646 95.203265)
+					(xy 131.152233 95.203265) (xy 131.152233 94.351346) (xy 132.184891 94.351346)
+				)
+			)
+			(polygon
+				(pts
+					(xy 133.199965 94.351346) (xy 133.828035 94.351346) (xy 133.828035 96.36) (xy 133.199965 96.36)
+				)
+			)
+			(polygon
+				(pts
+					(xy 135.598063 95.530429) (xy 136.148098 95.697247) (xy 136.102155 95.848004) (xy 136.043942 95.975267)
+					(xy 135.974319 96.082173) (xy 135.88893 96.176238) (xy 135.791643 96.252933) (xy 135.681228 96.313349)
+					(xy 135.56196 96.354597) (xy 135.415409 96.381507) (xy 135.236217 96.391263) (xy 135.018893 96.379314)
+					(xy 134.842756 96.346485) (xy 134.700837 96.296374) (xy 134.603862 96.242153) (xy 134.512068 96.169852)
+					(xy 134.424852 96.077487) (xy 134.342044 95.962372) (xy 134.278788 95.84103) (xy 134.231652 95.700814)
+					(xy 134.201779 95.538638) (xy 134.191224 95.35091) (xy 134.203388 95.148812) (xy 134.237767 94.975251)
+					(xy 134.292019 94.826022) (xy 134.364977 94.697573) (xy 134.456716 94.587163) (xy 134.566834 94.494431)
+					(xy 134.694044 94.420978) (xy 134.840897 94.36657) (xy 135.010729 94.332208) (xy 135.207519 94.320083)
+					(xy 135.399968 94.331162) (xy 135.560441 94.362034) (xy 135.693966 94.409952) (xy 135.804815 94.473346)
+					(xy 135.902934 94.556625) (xy 135.989734 94.661328) (xy 136.065449 94.790444) (xy 136.129413 94.947909)
+					(xy 135.575104 95.07113) (xy 135.542645 94.984339) (xy 135.514532 94.934965) (xy 135.45714 94.87249)
+					(xy 135.388869 94.826887) (xy 135.311095 94.798722) (xy 135.22254 94.78903) (xy 135.122321 94.799973)
+					(xy 135.037772 94.831258) (xy 134.965464 94.882564) (xy 134.903436 94.956214) (xy 134.860486 95.043698)
+					(xy 134.830734 95.169962) (xy 134.819295 95.347491) (xy 134.827659 95.521427) (xy 134.849545 95.648307)
+					(xy 134.880972 95.738413) (xy 134.919312 95.800439) (xy 134.973558 95.853081) (xy 135.037146 95.890717)
+					(xy 135.111939 95.914081) (xy 135.20068 95.922316) (xy 135.313717 95.910072) (xy 135.400203 95.876454)
+					(xy 135.466416 95.823276) (xy 135.517778 95.752408) (xy 135.56215 95.656771)
+				)
+			)
+		)
 	)
 	(gr_text "PICalculator v1.5\nDesigned by:\nKyle Schmerge\nMax Pastushkov\nhttps://github.com/kpzip/PICalculator\n"

Commit message: Update proj.kicad_pcb
Parts:
- D1, D10, D11, D12, D13, D14, D15, D16, D17, D18, D19, D2, D20, D21, D22, D23, D24, D25, D26, D27, D28, D29, D3, D30, D31, D32, D33, D34, D35, D36, D37, D38, D39, D4, D40, D41, D42, D5, D6, D7, D8, D9: value SMD1200PL-TP -> B5819W
