File: pcb/1.0/proj.kicad_pcb (KiCad board)
At the start: 2 copper layers, 125 x 185 mm, 115 parts, among them J1 Conn_01x04, SW1 Reset, SW10 8, SW11 9, SW12 /, SW13 Deg/Rad, SW14 Clear, SW15 4, SW16 5, SW17 6, SW18 X, SW19 Constants, SW2 Y/Stats, SW20 Del, SW21 1, SW22 2, SW23 3, SW24 -, SW25 Alpha, SW26 (/), SW27 Sin(x)/Sin-1(x), SW28 Cos(x)/Cos-1(x), SW29 Tan(x)/Tan-1(x), SW3 ./,, SW30 +, SW31 2nd, SW32 Γ(x), SW33 x^y/y√x, SW34 x^2/√x, SW35 log(x)/ln(x), SW36 e^x/10^x, SW37 Graph, SW38 Programs, SW39 Left, SW4 0, SW40 Up, SW41 Right, SW42 Down, SW43 Power, SW44 FPU Reset, SW45 Main Reset, SW5 +/-, SW6 Solve/=, SW7 Sci/Norm, SW8 X/Matrix, SW9 7, U1 PIC16C74, U2 STM32F401RCTx, U3 74HC238, U4 LTC3525-5, Y1 20MHz

Commit message: pcb work
Parts:
- removed SW45: Main Reset, Button_Switch_THT:SW_PUSH_6mm
- SW44: value FPU Reset -> Reset
- moved B2 4.50 mm to (137.8, 151.9), turned to 0 degrees
- moved B1 0.18 mm to (137.9, 132.0), turned to 0 degrees
Connections:
- C3 pad 1: +5V -> +3.3V
- C5 pad 1: +5V -> +3.3V
- C6 pad 1: +5V -> +3.3V
- DS1 pad 17: +5V -> +3.3V
- DS1 pad 2: +5V -> +3.3V
- RV1 pad 1: +5V -> +3.3V
- U1 pad 1: +5V -> +3.3V
- U1 pad 11: +5V -> +3.3V
- U1 pad 32: +5V -> +3.3V
- U2 pad 20: Net-(U2-PA4) -> COSS
- U2 pad 21: Net-(U2-PA5) -> SCK
- U2 pad 23: Net-(U2-PA7) -> MOSI
- U3 pad 16: +5V -> +3.3V
- U3 pad 6: +5V -> +3.3V
Routing:
- net +5V: track 246.7 -> 126.3 mm, vias 2 -> 1
- net +3.3V: track 51.7 -> 91.6 mm
- net Net-(B1-+): track 192.7 -> 198.7 mm
- net GND: track 52.7 -> 47.8 mm, vias 6 -> 2
Other:
- board text added: "PICalculator v1.0 Designed by: Kyle Schmerge Max Pastushkov Janet Shen https://github.com/kpzip/PICalculator"
- board text removed: "PICalculator v1.1 Designed by: Kyle Schmerge Max Pastushkov Janet Shen https://github.com/kpzip/PICalculator"
