File: pcb/1.0/proj.kicad_sch (KiCad schematic)
At the start: 123 parts, among them J1 Conn_01x04, SW1 Reset, SW10 8, SW11 9, SW12 /, SW13 Deg/Rad, SW14 Clear, SW15 4, SW16 5, SW17 6, SW18 X, SW19 Constants, SW2 Y/Stats, SW20 Del, SW21 1, SW22 2, SW23 3, SW24 -, SW25 Alpha, SW26 (/), SW27 Sin(x)/Sin-1(x), SW28 Cos(x)/Cos-1(x), SW29 Tan(x)/Tan-1(x), SW3 ./,, SW30 +, SW31 2nd, SW32 Γ(x), SW33 x^y/y√x, SW34 x^2/√x, SW35 log(x)/ln(x), SW36 e^x/10^x, SW37 Graph, SW38 Programs, SW39 Left, SW4 0, SW40 Up, SW41 Right, SW42 Down, SW43 Power, SW44 FPU Reset, SW45 Main Reset, SW5 +/-, SW6 Solve/=, SW7 Sci/Norm, SW8 X/Matrix, SW9 7, U1 PIC16C74, U2 STM32F401RCTx, U3 74HC238, U4 LTC3525-5, Y1 20MHz

Commit message: pcb work
Parts:
- removed R10, R6, R8: 20kΩ, symbol Device:R_US
- removed R11, R12, R5, R7, R9: 10kΩ, symbol Device:R_US
- removed SW45: Main Reset, Button_Switch_THT:SW_PUSH_6mm, symbol Switch:SW_Push
- SW44: value FPU Reset -> Reset
Connections:
- net +3.3V: now also C3.1, C5.1, C6.1, DS1.17 (~{RST}), DS1.2 (VDD), RV1.1, U1.1 (~{MCLR}/Vpp), U1.11 (VDD), U1.32 (VDD), U3.16 (VCC), U3.6 (E3)
- net +5V: no longer C3.1, C5.1, C6.1, DS1.17 (~{RST}), DS1.2 (VDD), RV1.1, U1.11 (VDD), U1.32 (VDD), U3.16 (VCC), U3.6 (E3)
- net COSS: now also U2.20 (PA4)
- net MOSI: now also U2.23 (PA7)
- net SCK: now also U2.21 (PA5)
Other:
- moved on the sheet: B1, B2, C3, J1, SW43

Commit message: add titles
Other:
- title: (none) -> PICalculator
Changed lines of the file:
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@@
 (kicad_sch
-	(version 20231120)
+	(version 20250114)
 	(generator "eeschema")
-	(generator_version "8.0")
+	(generator_version "9.0")
 	(paper "A3")
+	(title_block
+		(title "PICalculator")
+		(date "2025-02-05")
+		(rev "1.0")
+	)
 	(junction
 		(at 246.38 49.53)
@@
 		)
 	)
+	(embedded_fonts no)
 )
