File: pcb/1.1/proj.kicad_sch (KiCad schematic)
At the start: 125 parts, among them J1 Conn_02x05_Odd_Even, SW1 Reset, SW10 8, SW11 9, SW12 /, SW13 Deg/Rad, SW14 Clear, SW15 4, SW16 5, SW17 6, SW18 X, SW19 Constants, SW2 Y/Stats, SW20 Del, SW21 1, SW22 2, SW23 3, SW24 -, SW25 Alpha, SW26 (/), SW27 Sin(x)/Sin-1(x), SW28 Cos(x)/Cos-1(x), SW29 Tan(x)/Tan-1(x), SW3 ./,, SW30 +, SW31 2nd, SW32 Γ(x), SW33 x^y/y√x, SW34 x^2/√x, SW35 log(x)/ln(x), SW36 e^x/10^x, SW37 Graph, SW38 Programs, SW39 Left, SW4 0, SW40 Up, SW41 Right, SW42 Down, SW43 Power, SW44 FPU BOOT0, SW45 Reset, SW5 +/-, SW6 Solve/=, SW7 Sci/Norm, SW8 X/Matrix, SW9 7, U1 PIC16C74, U2 STM32F401RCTx, U3 74HC238, U4 ISL9111EH50Z-T7A, U5 SN74LVC1G32DBVR, Y1 20MHz

Commit message: add titles
Other:
- title: (none) -> PICalculator
Changed lines of the file:
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@@
 (kicad_sch
-	(version 20231120)
+	(version 20250114)
 	(generator "eeschema")
-	(generator_version "8.0")
+	(generator_version "9.0")
 	(paper "A3")
+	(title_block
+		(title "PICalculator")
+		(date "2025-03-05")
+		(rev "1.1")
+	)
 	(junction
 		(at 246.38 49.53)
@@
 		)
 	)
+	(embedded_fonts no)
 )
