File: pcb/1.2/proj.kicad_sch (KiCad schematic)
At the start: 128 parts, among them J1 Conn_02x05_Odd_Even, Q1 MMBT3904, SW1 Reset, SW10 8, SW11 9, SW12 /, SW13 Deg/Rad, SW14 Clear, SW15 4, SW16 5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

Commit message: add titles
Other:
- title: (none) -> PICalculator
Changed lines of the file:
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@@
 	(generator_version "9.0")
 	(paper "A3")
+	(title_block
+		(title "PICalculator")
+		(date "2025-05-08")
+		(rev "1.2")
+	)
 	(junction
 		(at 246.38 49.53)
